File: notiDroid-devBoard/devBoard-v1.sch (EAGLE design)
At the start: 0 parts

Commit message: WIP : first dev board
Parts:
- added C1, C2, C3: 1uF, rcl:C-EU050-024X044
- added C4, C6: 47pF, rcl:C-EU025-024X044
- added JP1, JP2: M14, SparkFun-Connectors:M14
- added JP3: M13, SparkFun-Connectors:M13
- added JP4: USB-B, SparkFun-Connectors:USBPTH
- added JP5: (no value), SparkFun-Connectors:M081X08
- added JP6: M09, SparkFun-Connectors:M09
- added R1, R2, R3: 33, rcl:R-EU_0207/10
- added U$1: LM1086, notiDroid-components:LM1086
- added U$2: PIC-ICSP-MINI, SparkFun-Connectors:PIC-ICSP-MINI
- added U$3: PIC18(L)F26K22, PIC18:PIC18(L)F26K22
- added U$4: BLE112", BLE112:BLE112"
Connections:
- new net AVDD: C1.1, C2.1, C3.1, JP3.11, JP3.12, JP3.5, JP5.2, U$4.AVDD@1, U$4.AVDD@2, U$4.DVDD, U$4.VDD_USB
- new net GND: C1.2, C2.2, C3.2, C4.1, C6.1, JP4.GND
- new net N$1: JP3.13, U$4.GND@1
- new net N$10: JP3.4, U$4.GND@2
- new net N$11: JP2.13, U$3.RA0
- new net N$12: JP2.12, U$3.RA1
- new net N$13: JP3.1, U$4.P1_5
- new net N$14: JP6.1, U$4.P$17
- new net N$15: JP6.2, U$4.RESET
- new net N$16: JP6.3, U$4.P0_0
- new net N$17: JP6.4, U$4.P0_1
- new net N$18: JP6.5, U$4.P0_2
- new net N$19: JP6.6, U$4.P0_3
- new net N$2: JP4.D-, R2.1
- new net N$20: JP6.7, U$4.P0_4
- new net N$21: JP6.8, U$4.P0_5
- new net N$22: JP6.9, U$4.P0_6
- new net N$23: JP5.7, U$4.P1_3
- new net N$24: JP5.8, U$4.P1_4
- new net N$25: JP5.6, U$4.P1_2
- new net N$26: JP5.5, U$4.P1_1
- new net N$27: JP2.11, U$3.RA2
- new net N$28: JP5.3, U$4.P0_7
- new net N$29: JP2.10, U$3.RA3
- new net N$3: JP4.D+, R1.1, R3.2
- new net N$30: JP5.1, U$4.GND@3
- new net N$31: JP2.9, U$3.RA4
- new net N$32: JP2.8, U$3.RA5
- new net N$33: JP2.7, U$3.VSS@1
- new net N$34: JP2.6, U$3.RA7
- new net N$35: JP2.5, U$3.RA6
- new net N$36: JP2.4, U$3.RC0
- new net N$37: JP2.3, U$3.RC1
- new net N$38: JP2.2, U$3.RC2
- new net N$39: JP2.1, U$3.RC3
- new net N$4: JP3.10, U$4.P2_2
- new net N$40: JP1.1, U$3.RB7
- new net N$41: JP1.2, U$3.RB6
- new net N$42: JP1.3, U$3.RB5
- new net N$43: JP1.4, U$3.RB4
- new net N$44: JP1.5, U$3.RB3
- new net N$45: JP1.6, U$3.RB2
- new net N$46: JP1.7, U$3.RB1
- new net N$47: JP1.8, U$3.RB0
- new net N$48: JP1.9, U$3.VDD
- new net N$49: JP1.10, U$3.VSS@2
- new net N$5: JP3.9, U$4.P2_1
- new net N$50: JP1.11, U$3.RC7
- new net N$51: JP1.12, U$3.RC6
- new net N$52: JP1.13, U$3.RC5
- new net N$53: JP1.14, U$3.RC4
- new net N$6: JP3.8, U$4.P2_0
- new net N$7: JP3.7, U$4.P1_7
- new net N$8: JP3.6, U$4.P1_6
- new net N$9: JP2.14, U$3.MCLR
- new net P1_0: JP5.4, R3.1, U$4.P1_0
- new net USB+: C6.2, JP3.3, R1.2, U$4.USB+
- new net USB-: C4.2, JP3.2, R2.2, U$4.USB-
